File: Kicad/esp32-s3 single motor & battery controller/PSU.kicad_sch (KiCad schematic)
At the start: 72 parts, among them J5 JST XH-S, Q1 PJA3430, Q2 PJA3430, Q3 Vishay sir404dp, Q4 PJA3430, Q5 PJA3430, Q7 Vishay sir404dp, U2 AP63203WU, U3 BQ76905RGRR, U4 BQ24780SRUYR

Commit message: Gerbers and BOM for v0.4 PCB
I adjusted all the testpoints to be excluded from the BOM.
Parts:
- TP6: now left out of the parts list
Changed lines of the file:
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@@
 		(unit 1)
 		(exclude_from_sim no)
-		(in_bom yes)
+		(in_bom no)
 		(on_board yes)
 		(dnp no)
